File: pa-jtag.kicad_sch (KiCad schematic)
At the start: 67 parts, among them J1 USB_B, J2 RS232, J3 VCCIO, J4 VOUT, U2 L78L33_TO92

Commit message: ch32v103c schematic / placement
Parts:
- removed J3: VCCIO, Connector_PinHeader_2.54mm:PinHeader_1x03_P2.54mm_Horizontal, symbol Connector:Conn_01x03_Male
- removed J?: UART, symbol Connector:Conn_01x03_Male
- removed J?: I2C, symbol Connector:Conn_01x03_Male
- removed J?: SWD, symbol Connector:Conn_01x06_Male
- removed R?: 0R, symbol Device:R
- added J: Conn_02x03_Odd_Even, symbol Connector_Generic:Conn_02x03_Odd_Even
- added J: Conn_02x06_Odd_Even, symbol Connector_Generic:Conn_02x06_Odd_Even
- added SW: SW_Push_45deg, symbol Switch:SW_Push_45deg
- added U: (no value), symbol Device:CP
- added U: (no value), symbol Device:R
- added U (x2): (no value), symbol Device:C
- U: renamed from D3; value NUP2105L -> (none); footprint Package_TO_SOT_SMD:SOT-23 -> (none)
- U: renamed from J1; value USB_B -> (none); footprint Connector_USB:USB_Mini-B_Wuerth_65100516121_Horizontal -> (none)
- U: renamed from D4; value NUP2105L -> (none); footprint Package_TO_SOT_SMD:SOT-23 -> (none)
- U: renamed from D1; value VBUS -> (none); footprint LED_SMD:LED_0603_1608Metric -> (none)
- U: renamed from R1; value 470 -> (none); footprint Resistor_SMD:R_0603_1608Metric -> (none)
- U: renamed from L1; value 10uH -> (none); footprint Inductor_SMD:L_0805_2012Metric -> (none)
- U: renamed from D2; value NUP2105L -> (none); footprint Package_TO_SOT_SMD:SOT-23 -> (none)
- U: renamed from C1; value 10nF -> (none); footprint Capacitor_SMD:C_0603_1608Metric -> (none)
- U: renamed from C3; value 100nF -> (none); footprint Capacitor_SMD:C_0603_1608Metric -> (none)
- U: renamed from C4; value 100nF -> (none); footprint Capacitor_SMD:C_0603_1608Metric -> (none)
- U: renamed from C2; value 6.8uF -> (none); footprint Capacitor_Tantalum_SMD:CP_EIA-3216-18_Kemet-A -> (none)
- U: renamed from R2; value 10R -> (none); footprint Resistor_SMD:R_0603_1608Metric -> (none)
- U: renamed from R3; value 10R -> (none); footprint Resistor_SMD:R_0603_1608Metric -> (none)
- U: renamed from R4; value 10R -> (none); footprint Resistor_SMD:R_0603_1608Metric -> (none)
- U: renamed from R6; value 10R -> (none); footprint Resistor_SMD:R_0603_1608Metric -> (none)
- U: renamed from R7; value 10R -> (none); footprint Resistor_SMD:R_0603_1608Metric -> (none)
- U: renamed from D?; value NUP2105L -> (none); footprint Package_TO_SOT_SMD:SOT-23 -> (none)
- U: renamed from R?; value 470 -> (none); footprint Resistor_SMD:R_0603_1608Metric -> (none)
- U: renamed from R9; value 10R -> (none); footprint Resistor_SMD:R_0603_1608Metric -> (none)
- U: renamed from U?; value MAX3232 -> (none)
- U: renamed from D?; value ST1 -> (none); footprint LED_SMD:LED_0603_1608Metric -> (none)
- U: renamed from D5; value 1N4148 -> (none); footprint Diode_SMD:D_MiniMELF -> (none)
- U: renamed from R?; value 100R -> (none)
- U: renamed from R12; value 10K -> (none); footprint Resistor_SMD:R_0603_1608Metric -> (none)
- U: renamed from C?; value 100nF -> (none); footprint Capacitor_SMD:C_0603_1608Metric -> (none)
- U: renamed from C?; value 100nF -> (none)
- U: renamed from R?; value 4K7 -> (none)
- U: renamed from R5; value 10R -> (none); footprint Resistor_SMD:R_0603_1608Metric -> (none)
- U: renamed from J4; value VOUT -> (none); footprint Connector_PinHeader_2.54mm:PinHeader_1x03_P2.54mm_Horizontal -> (none)
- U: renamed from D?; value 1N4148 -> (none); footprint Diode_SMD:D_MiniMELF -> (none)
- U: renamed from J?; value CH_SWD -> (none)
- U: renamed from R?; value 10R -> (none); footprint Resistor_SMD:R_0603_1608Metric -> (none)
- U: renamed from J?; value AUX -> (none)
- U: renamed from C?; value 20pF -> (none)
- U: renamed from J2; value RS232 -> (none); footprint Connector_Dsub:DSUB-9_Female_Horizontal_P2.77x2.84mm_EdgePinOffset7.70mm_Housed_MountingHolesOffset9.12mm -> (none)
- U: renamed from R?; value 10K -> (none); footprint Resistor_SMD:R_0603_1608Metric -> (none)
- U: renamed from U?; value CH32V103C8T6 -> (none); footprint Package_QFP:LQFP-48_7x7mm_P0.5mm -> (none)
- U: renamed from U2; value L78L33_TO92 -> (none); footprint Package_TO_SOT_THT:TO-92_Inline -> (none)
- U: renamed from R8; value 10R -> (none); footprint Resistor_SMD:R_0603_1608Metric -> (none)
- U: renamed from D?; value ST0 -> (none); footprint LED_SMD:LED_0603_1608Metric -> (none)
- U: renamed from J?; value JTAG -> (none)
- U: renamed from R?; value 10K -> (none)
- U: renamed from R13; value 10K -> (none); footprint Resistor_SMD:R_0603_1608Metric -> (none)
- U: renamed from Y?; value 8M -> (none)
Connections:
- net +VSW: now also J.3 (Pin_3), U.1
- net BOOT1: now also U.1
- net CH_NRST: now also SW.1
- net GND: now also U.1, J.12 (Pin_12), J.5 (Pin_5), J.6 (Pin_6), SW.2, U.1, U.2, U.2, U.2
- net I2C_SCL: now also J.8 (Pin_8)
- net I2C_SDA: now also J.10 (Pin_10)
- net MCU-SRST: now also U.1 (K); no longer U.2 (K)
- net MCU-TDI: now also U.1 (K); no longer U.2 (K)
- net MCU-TDO: now also U.2 (K); no longer U.1 (K)
- net MCU-TRST: now also U.2 (K); no longer U.1 (K)
- net NRST: now also J.9 (Pin_9)
- net SWCLK: now also J.3 (Pin_3)
- net SWDIO: now also J.7 (Pin_7)
- net SWO: now also J.11 (Pin_11)
- net UART_RX: now also J.4 (Pin_4)
- net UART_TX: now also J.2 (Pin_2)
- net VOUT: now also J.1 (Pin_1)
- net VOUTR: now also J.2 (Pin_2)
- net VTARGET: now also J.5 (Pin_5), J.6 (Pin_6)
- net at U.2, U.2 (D-): now also U.2 (K); no longer U.1 (K)
- net at U.2, U.3 (D+): now also U.1 (K); no longer U.2 (K)
- net at U.2 (VS+): now also U.2; no longer U.1
- net at U.6 (VS-): now also U.2; no longer U.2
- net ST0: now reaches U.2 (A)
- net ST0: now also U.3 (PC14)
- net ST1: now reaches U.4 (PC15)
- net ST1: now also U.2 (A)
- new net VSWD: J.1 (Pin_1), J.4 (Pin_4), U.1
- no-connect marks 4 -> 5
Other:
- company: (C) 2022 Pike Aerospace Research Corporation -> (C) 2022 Mike Sharkey (mike@8bitgeek.net)
- title: HIGH SPEED USB TO JTAG / SWD / UART / I2S / GPIO -> Bug-O-Matic  - JTAG / SWD / UART / I2S / GPIO
- moved on the sheet: U
